File: Schematic/Borjomi.sch (KiCad schematic (older format))
At the start: 10 parts, among them J1 Vin 12V, J2 Vout 12V, J3 Water Switch 12V, J4 Data in, J5 Data out, J6 Conn_01x02, K1 SRD-5VDC-SL-C, U1 MCP2515-TJA1050, U2 MH-Series

Commit message: Add relay module (scheme, lib, footprint)
Parts:
- removed K1: SRD-5VDC-SL-C, Relay_THT:Relay_SPDT_SANYOU_SRD_Series_Form_C, symbol Relay:SANYOU_SRD_Form_C
- added U3: 5V_Relay_Module, RelayModule:Relay_Module_1_Channel, symbol RelayModule:5V_1_Channel_Relay_Module
- J1, J2, J3, J6: footprint (none) -> Connector_Wire:SolderWirePad_1x02_P5.08mm_Drill1.5mm
- J4, J5: footprint (none) -> Connector_RJ:RJ12_Amphenol_54601
Connections:
- net labels added: +12V
- wire segments 78 -> 86
- no-connect marks 0 -> 21
Other:
- moved on the sheet: J3
Changed lines of the file:
@@
 EESchema Schematic File Version 4
-EELAYER 26 0
+LIBS:Borjomi-cache
+EELAYER 29 0
 EELAYER END
 $Descr A4 11693 8268
@@
 Wire Wire Line
 	4750 1750 6200 1750
-Wire Wire Line
-	7600 4150 7600 2800
 $Comp
 L Connector:Screw_Terminal_01x02 J1
@@
 F 0 "J1" H 1470 1525 50  0000 C CNN
 F 1 "Vin 12V" H 1470 1616 50  0000 C CNN
-F 2 "" H 1550 1850 50  0001 C CNN
+F 2 "Connector_Wire:SolderWirePad_1x02_P5.08mm_Drill1.5mm" H 1550 1850 50  0001 C CNN
 F 3 "~" H 1550 1850 50  0001 C CNN
 	1    1550 1850
@@
 F 0 "J2" H 1470 1975 50  0000 C CNN
 F 1 "Vout 12V" H 1470 2066 50  0000 C CNN
-F 2 "" H 1550 2300 50  0001 C CNN
+F 2 "Connector_Wire:SolderWirePad_1x02_P5.08mm_Drill1.5mm" H 1550 2300 50  0001 C CNN
 F 3 "~" H 1550 2300 50  0001 C CNN
 	1    1550 2300
 	-1   0    0    1
 $EndComp
-Wire Wire Line
-	4650 3750 4650 4150
-Wire Wire Line
-	4650 4150 7600 4150
 $Comp
 L power:GND #PWR04
@@
 $EndComp
 Wire Wire Line
-	4550 3750 4550 3900
+	4550 3750 4550 3850
 $Comp
 L power:GND #PWR01
@@
 F 0 "J4" H 1470 3675 50  0000 C CNN
 F 1 "Data in" H 1470 3766 50  0000 C CNN
-F 2 "" H 1550 4100 50  0001 C CNN
+F 2 "Connector_RJ:RJ12_Amphenol_54601" H 1550 4100 50  0001 C CNN
 F 3 "~" H 1550 4100 50  0001 C CNN
 	1    1550 4100
@@
 F 0 "J5" H 1470 2825 50  0000 C CNN
 F 1 "Data out" H 1470 2916 50  0000 C CNN
-F 2 "" H 1550 3250 50  0001 C CNN
+F 2 "Connector_RJ:RJ12_Amphenol_54601" H 1550 3550 50  0001 C CNN
 F 3 "~" H 1550 3250 50  0001 C CNN
 	1    1550 3250
@@
 	1900 4800 1900 4300
 Connection ~ 1900 4300
-$Comp
-L Relay:SANYOU_SRD_Form_C K1
-U 1 1 5B6FFEB6
-P 2900 2850
-F 0 "K1" H 2470 2804 50  0000 R CNN
-F 1 "SRD-5VDC-SL-C" H 2470 2895 50  0000 R CNN
-F 2 "Relay_THT:Relay_SPDT_SANYOU_SRD_Series_Form_C" H 3350 2800 50  0001 L CNN
-F 3 "http://www.sanyourelay.ca/public/products/pdf/SRD.pdf" H 2900 2850 50  0001 C CNN
-	1    2900 2850
-	-1   0    0    1
-$EndComp
 Wire Wire Line
 	2100 1750 2400 1750
@@
 L power:GND #PWR03
 U 1 1 5B7075AE
-P 3100 3500
-F 0 "#PWR03" H 3100 3250 50  0001 C CNN
-F 1 "GND" H 3105 3327 50  0000 C CNN
-F 2 "" H 3100 3500 50  0001 C CNN
-F 3 "" H 3100 3500 50  0001 C CNN
-	1    3100 3500
-	1    0    0    -1
-$EndComp
-Wire Wire Line
-	3100 3150 3100 3500
-Wire Wire Line
-	3100 2550 3100 2450
-Wire Wire Line
-	3100 2450 4050 2450
+P 3500 3350
+F 0 "#PWR03" H 3500 3100 50  0001 C CNN
+F 1 "GND" H 3505 3177 50  0000 C CNN
+F 2 "" H 3500 3350 50  0001 C CNN
+F 3 "" H 3500 3350 50  0001 C CNN
+	1    3500 3350
+	1    0    0    -1
+$EndComp
+Wire Wire Line
+	3300 2700 3300 2450
+Wire Wire Line
+	3300 2450 4050 2450
 $Comp
 L Connector:Screw_Terminal_01x02 J3
 U 1 1 5B709E73
-P 2700 1100
-F 0 "J3" V 2700 900 50  0000 C CNN
-F 1 "Water Switch 12V" V 2550 600 50  0000 C CNN
-F 2 "" H 2700 1100 50  0001 C CNN
-F 3 "~" H 2700 1100 50  0001 C CNN
-	1    2700 1100
+P 2600 1250
+F 0 "J3" V 2600 1050 50  0000 C CNN
+F 1 "Water Switch 12V" V 2450 750 50  0000 C CNN
+F 2 "Connector_Wire:SolderWirePad_1x02_P5.08mm_Drill1.5mm" H 2600 1250 50  0001 C CNN
+F 3 "~" H 2600 1250 50  0001 C CNN
+	1    2600 1250
 	0    -1   -1   0
 $EndComp
@@
 L power:GND #PWR02
 U 1 1 5B70B3E3
-P 2800 1400
-F 0 "#PWR02" H 2800 1150 50  0001 C CNN
-F 1 "GND" H 2805 1227 50  0000 C CNN
-F 2 "" H 2800 1400 50  0001 C CNN
-F 3 "" H 2800 1400 50  0001 C CNN
-	1    2800 1400
-	1    0    0    -1
-$EndComp
-Wire Wire Line
-	2800 1300 2800 1400
-Wire Wire Line
-	2700 1300 2700 2550
-Wire Wire Line
-	2400 1750 2400 3400
-Wire Wire Line
-	2400 3400 2600 3400
-Wire Wire Line
-	2600 3400 2600 3150
+P 2700 1550
+F 0 "#PWR02" H 2700 1300 50  0001 C CNN
+F 1 "GND" H 2705 1377 50  0000 C CNN
+F 2 "" H 2700 1550 50  0001 C CNN
+F 3 "" H 2700 1550 50  0001 C CNN
+	1    2700 1550
+	1    0    0    -1
+$EndComp
+Wire Wire Line
+	2700 1450 2700 1550
+Wire Wire Line
+	2600 1450 2600 2700
+Wire Wire Line
+	2400 1750 2400 2800
 Connection ~ 2400 1750
 Wire Wire Line
@@
 F 0 "J6" H 8530 1192 50  0000 L CNN
 F 1 "Conn_01x02" H 8530 1101 50  0000 L CNN
-F 2 "" H 8450 1200 50  0001 C CNN
+F 2 "Connector_Wire:SolderWirePad_1x02_P5.08mm_Drill1.5mm" H 8450 1200 50  0001 C CNN
 F 3 "~" H 8450 1200 50  0001 C CNN
 	1    8450 1200
@@
 Wire Wire Line
 	8250 1300 7000 1300
+NoConn ~ 2600 2900
+NoConn ~ 4050 2150
+NoConn ~ 4050 2650
+NoConn ~ 4050 2250
+NoConn ~ 4050 2550
+NoConn ~ 4050 2750
+NoConn ~ 4050 2850
+NoConn ~ 4050 2950
+NoConn ~ 4050 3150
+NoConn ~ 5050 3450
+NoConn ~ 5050 3350
+NoConn ~ 5050 3250
+NoConn ~ 5050 3150
+NoConn ~ 5050 3050
+NoConn ~ 5050 2950
+NoConn ~ 5050 2850
+NoConn ~ 5050 2550
+NoConn ~ 5050 2250
+NoConn ~ 5050 2150
+NoConn ~ 4650 1750
+NoConn ~ 6200 1100
+$Comp
+L power:+12V #PWR0101
+U 1 1 5C9D63F0
+P 2100 1450
+F 0 "#PWR0101" H 2100 1300 50  0001 C CNN
+F 1 "+12V" H 2115 1623 50  0000 C CNN
+F 2 "" H 2100 1450 50  0001 C CNN
+F 3 "" H 2100 1450 50  0001 C CNN
+	1    2100 1450
+	1    0    0    -1
+$EndComp
+Wire Wire Line
+	2100 1450 2100 1750
+$Comp
+L power:GND #PWR0102
+U 1 1 5C9DAC98
+P 7600 2950
+F 0 "#PWR0102" H 7600 2700 50  0001 C CNN
+F 1 "GND" H 7605 2777 50  0000 C CNN
+F 2 "" H 7600 2950 50  0001 C CNN
+F 3 "" H 7600 2950 50  0001 C CNN
+	1    7600 2950
+	1    0    0    -1
+$EndComp
+Wire Wire Line
+	7600 2800 7600 2950
+Wire Wire Line
+	4650 3750 4650 3850
+Wire Wire Line
+	4650 3850 4550 3850
+Connection ~ 4550 3850
+Wire Wire Line
+	4550 3850 4550 3900
+$Comp
+L power:PWR_FLAG #FLG0101
+U 1 1 5C9DFAE5
+P 4350 3900
+F 0 "#FLG0101" H 4350 3975 50  0001 C CNN
+F 1 "PWR_FLAG" H 4450 4100 50  0000 C CNN
+F 2 "" H 4350 3900 50  0001 C CNN
+F 3 "~" H 4350 3900 50  0001 C CNN
+	1    4350 3900
+	-1   0    0    1
+$EndComp
+Wire Wire Line
+	4350 3850 4550 3850
+Wire Wire Line
+	4350 3900 4350 3850
+$Comp
+L RelayModule:5V_1_Channel_Relay_Module U3
+U 1 1 5CA61D0C
+P 2950 2800
+F 0 "U3" H 2950 3150 50  0000 C CNN
+F 1 "5V_Relay_Module" H 2950 3050 50  0000 C CNN
+F 2 "RelayModule:Relay_Module_1_Channel" H 2950 2800 50  0001 C CNN
+F 3 "http://arduino.ua/prod2888-modyl-rele-5v-10a-visokogo-yrovnya-high-level" H 2950 2800 50  0001 C CNN
+	1    2950 2800
+	-1   0    0    1
+$EndComp
+Wire Wire Line
+	2400 2800 2600 2800
+Wire Wire Line
+	3300 2800 3500 2800
+Wire Wire Line
+	3500 2800 3500 3350
+Wire Wire Line
+	4750 1750 4750 1600
+Wire Wire Line
+	4750 1600 3400 1600
+Wire Wire Line
+	3400 1600 3400 2900
+Wire Wire Line
+	3400 2900 3300 2900
+Connection ~ 4750 1750
 $EndSCHEMATC

Commit message: Add footprints for components; add pcb basic
Parts:
- J4, J5: footprint Connector_RJ:RJ12_Amphenol_54601 -> Connector:RJ14_YH-57-21_5722_6P4C; symbol Connector_Generic:Conn_01x05 -> Connector:RJ14
- U1: footprint Package_SO:TSSOP-20_4.4x6.5mm_P0.65mm -> CAN:AOC346_MCP2515
- U2: footprint Package_DFN_QFN:AMS_QFN-4-1EP_2x2mm_P0.95mm_EP0.7x1.6mm -> MH_Sensor:MH_Sensor
Connections:
- net labels removed: shield
- wire segments 86 -> 85
Changed lines of the file:
@@
 F 0 "U1" H 7600 3128 50  0000 C CNN
 F 1 "MCP2515-TJA1050" H 7600 3037 50  0000 C CNN
-F 2 "Package_SO:TSSOP-20_4.4x6.5mm_P0.65mm" H 7600 1450 50  0001 C CIN
-F 3 "http://ww1.microchip.com/downloads/en/DeviceDoc/21801e.pdf" H 7700 1550 50  0001 C CNN
+F 2 "CAN:AOC346_MCP2515" H 7600 1450 50  0001 C CIN
+F 3 "http://arduino.ua/prod1347-modyl-can-shini-na-mcp2515-i-tja1050" H 7700 1550 50  0001 C CNN
 	1    7600 2350
 	1    0    0    -1
@@
 	2100 1750 1750 1750
 $Comp
-L Connector_Generic:Conn_01x05 J4
+L Connector:RJ14 J4
 U 1 1 5B6F8A1D
-P 1550 4100
-F 0 "J4" H 1470 3675 50  0000 C CNN
-F 1 "Data in" H 1470 3766 50  0000 C CNN
-F 2 "Connector_RJ:RJ12_Amphenol_54601" H 1550 4100 50  0001 C CNN
-F 3 "~" H 1550 4100 50  0001 C CNN
-	1    1550 4100
-	-1   0    0    1
-$EndComp
-$Comp
-L Connector_Generic:Conn_01x05 J5
+P 1350 4200
+F 0 "J4" H 1100 3850 50  0000 C CNN
+F 1 "Data in" H 1500 3850 50  0000 C CNN
+F 2 "Connector:RJ14_YH-57-21_5722_6P4C" H 1350 4200 50  0001 C CNN
+F 3 "https://www.rcscomponents.kiev.ua/product/rozetka-yh-57-21-5722-6p4c_12940.html" H 1350 4200 50  0001 C CNN
+	1    1350 4200
+	1    0    0    -1
+$EndComp
+$Comp
+L Connector:RJ14 J5
 U 1 1 5B6F8AB0
-P 1550 3250
-F 0 "J5" H 1470 2825 50  0000 C CNN
-F 1 "Data out" H 1470 2916 50  0000 C CNN
-F 2 "Connector_RJ:RJ12_Amphenol_54601" H 1550 3550 50  0001 C CNN
-F 3 "~" H 1550 3250 50  0001 C CNN
-	1    1550 3250
-	-1   0    0    1
+P 1350 3350
+F 0 "J5" H 1100 3000 50  0000 C CNN
+F 1 "Data out" H 1500 3000 50  0000 C CNN
+F 2 "Connector:RJ14_YH-57-21_5722_6P4C" H 1350 3650 50  0001 C CNN
+F 3 "https://www.rcscomponents.kiev.ua/product/rozetka-yh-57-21-5722-6p4c_12940.html" H 1350 3350 50  0001 C CNN
+	1    1350 3350
+	1    0    0    -1
 $EndComp
 Wire Wire Line
@@
 	1750 4200 1950 4200
 Wire Wire Line
-	1950 4200 1950 3350
-Wire Wire Line
 	1950 3350 1750 3350
 Wire Wire Line
-	1750 4100 2000 4100
-Wire Wire Line
 	2000 4100 2000 3250
 Wire Wire Line
-	2000 3250 1750 3250
-Wire Wire Line
-	1750 4000 2050 4000
-Wire Wire Line
 	2050 4000 2050 3150
-Wire Wire Line
-	2050 3150 1750 3150
-Wire Wire Line
-	1750 3900 2100 3900
-Wire Wire Line
-	2100 3900 2100 3050
-Wire Wire Line
-	2100 3050 1750 3050
-Text Label 1800 3050 0    50   ~ 0
-shield
 Wire Wire Line
 	1950 4200 1950 4750
@@
 F 0 "U2" H 6600 1525 50  0000 C CNN
 F 1 "MH-Series" H 6600 1434 50  0000 C CNN
-F 2 "Package_DFN_QFN:AMS_QFN-4-1EP_2x2mm_P0.95mm_EP0.7x1.6mm" H 6600 750 50  0001 C CNN
+F 2 "MH_Sensor:MH_Sensor" H 6600 750 50  0001 C CNN
 F 3 "https://ru.aliexpress.com/item/1pcs-lot-soil-the-hygrometer-detection-module-soil-moisture-sensor-Robot-smart-car/32826425650.html?spm=a2g0v.10010108.1000016.1.7ca9471dkqoaPU&isOrigTitle=true" H 6500 1150 50  0001 C CNN
 	1    6600 1150
@@
 	3400 2900 3300 2900
 Connection ~ 4750 1750
+Wire Wire Line
+	1750 3250 2000 3250
+Wire Wire Line
+	1750 3150 2050 3150
+Wire Wire Line
+	1950 4100 1950 4200
+Wire Wire Line
+	1950 4000 1950 4100
+Wire Wire Line
+	1950 3350 1950 4000
+Wire Wire Line
+	1750 4000 2050 4000
+Wire Wire Line
+	1750 4100 2000 4100
 $EndSCHEMATC

Commit message: Update footprints (place pads in right order)
Parts:
- U2: symbol Sensors:MH-Series -> Borjomi-rescue:MH-Series-Sensors
Connections:
- net at U2.5 (S+): now also J6.2 (Pin_2); no longer J6.1 (Pin_1)
- net at U2.6 (S-): now also J6.1 (Pin_1); no longer J6.2 (Pin_2)
Changed lines of the file:
@@
 	2400 1750 4450 1750
 $Comp
-L Sensors:MH-Series U2
+L Borjomi-rescue:MH-Series-Sensors U2
 U 1 1 5B713FC4
 P 6600 1150

Commit message: Pcb v1.0 + gerber files
Parts:
- added D1: 1N5408, Diode_THT:D_DO-27_P5.08mm_Vertical_KathodeUp, symbol Diode:1N5408
- J1, J2, J3, J6: footprint Connector_Wire:SolderWirePad_1x02_P5.08mm_Drill1.5mm -> Connector:Degson_DG301_1x02_P5.00mm_Horizontal
Connections:
- net +12V: now also U3.4 (NO); no longer U3.5 (COM)
- net GND: now also J3.1 (Pin_1), D1.2 (A); no longer J3.2 (Pin_2)
- net at A1.5 (D2): no longer U1.3 (~INT)
- net at A1.8 (D5): now also U1.3 (~INT)
- net at J4.2, J5.2: now also U1.2 (CAN_HI); no longer U1.1 (CAN_LO)
- net at J4.1, J5.1: now also U1.1 (CAN_LO); no longer U1.2 (CAN_HI)
- net at U2.5 (S+): now also J6.1 (Pin_1); no longer J6.2 (Pin_2)
- net at U2.6 (S-): now also J6.2 (Pin_2); no longer J6.1 (Pin_1)
- new net: D1.1 (K), J3.2 (Pin_2), U3.5 (COM)
Other:
- moved on the sheet: J3
Changed lines of the file:
@@
 $EndComp
-Wire Wire Line
-	3850 1450 3850 2350
-Wire Wire Line
-	3850 2350 4050 2350
 Wire Wire Line
 	7000 2200 5800 2200
@@
 F 0 "J1" H 1470 1525 50  0000 C CNN
 F 1 "Vin 12V" H 1470 1616 50  0000 C CNN
-F 2 "Connector_Wire:SolderWirePad_1x02_P5.08mm_Drill1.5mm" H 1550 1850 50  0001 C CNN
+F 2 "Connector:Degson_DG301_1x02_P5.00mm_Horizontal" H 1550 1850 50  0001 C CNN
 F 3 "~" H 1550 1850 50  0001 C CNN
 	1    1550 1850
@@
 F 0 "J2" H 1470 1975 50  0000 C CNN
 F 1 "Vout 12V" H 1470 2066 50  0000 C CNN
-F 2 "Connector_Wire:SolderWirePad_1x02_P5.08mm_Drill1.5mm" H 1550 2300 50  0001 C CNN
+F 2 "Connector:Degson_DG301_1x02_P5.00mm_Horizontal" H 1550 2300 50  0001 C CNN
 F 3 "~" H 1550 2300 50  0001 C CNN
 	1    1550 2300
@@
 Wire Wire Line
 	1950 4200 1950 4750
-Wire Wire Line
-	8200 4750 8200 2600
 Connection ~ 1950 4200
 Wire Wire Line
-	8200 2500 8300 2500
-Wire Wire Line
-	8300 2500 8300 4800
-Wire Wire Line
-	1900 4800 1900 4300
+	8200 2600 8200 4650
 Connection ~ 1900 4300
-Wire Wire Line
-	2100 1750 2400 1750
 Connection ~ 2100 1750
 Wire Wire Line
-	1950 4750 8200 4750
-Wire Wire Line
-	1900 4800 8300 4800
+	1900 4650 8200 4650
 $Comp
 L power:GND #PWR03
@@
 L Connector:Screw_Terminal_01x02 J3
 U 1 1 5B709E73
-P 2600 1250
-F 0 "J3" V 2600 1050 50  0000 C CNN
-F 1 "Water Switch 12V" V 2450 750 50  0000 C CNN
-F 2 "Connector_Wire:SolderWirePad_1x02_P5.08mm_Drill1.5mm" H 2600 1250 50  0001 C CNN
-F 3 "~" H 2600 1250 50  0001 C CNN
-	1    2600 1250
-	0    -1   -1   0
+P 2500 1100
+F 0 "J3" V 2450 1200 50  0000 C CNN
+F 1 "Water Switch 12V" V 2350 1500 50  0000 C CNN
+F 2 "Connector:Degson_DG301_1x02_P5.00mm_Horizontal" H 2500 1100 50  0001 C CNN
+F 3 "~" H 2500 1100 50  0001 C CNN
+	1    2500 1100
+	0    1    -1   0
 $EndComp
 $Comp
 L power:GND #PWR02
 U 1 1 5B70B3E3
-P 2700 1550
-F 0 "#PWR02" H 2700 1300 50  0001 C CNN
-F 1 "GND" H 2705 1377 50  0000 C CNN
-F 2 "" H 2700 1550 50  0001 C CNN
-F 3 "" H 2700 1550 50  0001 C CNN
-	1    2700 1550
-	1    0    0    -1
-$EndComp
-Wire Wire Line
-	2700 1450 2700 1550
-Wire Wire Line
-	2600 1450 2600 2700
-Wire Wire Line
-	2400 1750 2400 2800
-Connection ~ 2400 1750
-Wire Wire Line
-	2400 1750 4450 1750
+P 2500 1400
+F 0 "#PWR02" H 2500 1150 50  0001 C CNN
+F 1 "GND" H 2505 1227 50  0000 C CNN
+F 2 "" H 2500 1400 50  0001 C CNN
+F 3 "" H 2500 1400 50  0001 C CNN
+	1    2500 1400
+	1    0    0    -1
+$EndComp
+Wire Wire Line
+	2500 1300 2500 1400
 $Comp
 L Borjomi-rescue:MH-Series-Sensors U2
@@
 Wire Wire Line
 	5600 1000 6200 1000
-$Comp
-L Connector_Generic:Conn_01x02 J6
-U 1 1 5B71928D
-P 8450 1200
-F 0 "J6" H 8530 1192 50  0000 L CNN
-F 1 "Conn_01x02" H 8530 1101 50  0000 L CNN
-F 2 "Connector_Wire:SolderWirePad_1x02_P5.08mm_Drill1.5mm" H 8450 1200 50  0001 C CNN
-F 3 "~" H 8450 1200 50  0001 C CNN
-	1    8450 1200
-	1    0    0    -1
-$EndComp
 Wire Wire Line
 	7000 1200 8250 1200
@@
 NoConn ~ 2600 2900
 NoConn ~ 4050 2150
-NoConn ~ 4050 2650
+NoConn ~ 4050 2350
 NoConn ~ 4050 2250
 NoConn ~ 4050 2550
@@
 $EndComp
 Wire Wire Line
-	2400 2800 2600 2800
-Wire Wire Line
 	3300 2800 3500 2800
 Wire Wire Line
@@
 Wire Wire Line
 	1750 4100 2000 4100
+$Comp
+L Connector_Generic:Conn_01x02 J6
+U 1 1 5B71928D
+P 8450 1300
+F 0 "J6" H 8530 1292 50  0000 L CNN
+F 1 "Conn_01x02" H 8530 1201 50  0000 L CNN
+F 2 "Connector:Degson_DG301_1x02_P5.00mm_Horizontal" H 8450 1300 50  0001 C CNN
+F 3 "~" H 8450 1300 50  0001 C CNN
+	1    8450 1300
+	1    0    0    1
+$EndComp
+Wire Wire Line
+	2600 1750 2600 2700
+Connection ~ 2600 1750
+Wire Wire Line
+	2600 1750 4450 1750
+Wire Wire Line
+	2100 1750 2600 1750
+Wire Wire Line
+	2400 2800 2600 2800
+Wire Wire Line
+	2400 1300 2400 2800
+Wire Wire Line
+	1900 4650 1900 4300
+Wire Wire Line
+	8300 2500 8300 4750
+Wire Wire Line
+	8200 2500 8300 2500
+Wire Wire Line
+	1950 4750 8300 4750
+Wire Wire Line
+	3850 2650 4050 2650
+Wire Wire Line
+	3850 1450 3850 2650
+$Comp
+L Diode:1N5408 D1
+U 1 1 5CAC420C
+P 2400 2950
+F 0 "D1" V 2400 2750 50  0000 L CNN
+F 1 "1N5408" V 2500 2650 50  0000 L CNN
+F 2 "Diode_THT:D_DO-27_P5.08mm_Vertical_KathodeUp" H 2400 2775 50  0001 C CNN
+F 3 "http://www.vishay.com/docs/88516/1n5400.pdf" H 2400 2950 50  0001 C CNN
+	1    2400 2950
+	0    1    1    0
+$EndComp
+Connection ~ 2400 2800
+$Comp
+L power:GND #PWR06
+U 1 1 5CAC8B8C
+P 2400 3100
+F 0 "#PWR06" H 2400 2850 50  0001 C CNN
+F 1 "GND" H 2405 2927 50  0000 C CNN
+F 2 "" H 2400 3100 50  0001 C CNN
+F 3 "" H 2400 3100 50  0001 C CNN
+	1    2400 3100
+	1    0    0    -1
+$EndComp
 $EndSCHEMATC

Commit message: PCB v1.1 + gerber
Parts:
- A1: footprint Module:Arduino_Nano -> Arduino:Arduino_Nano_Holes0.9
- U1: footprint CAN:AOC346_MCP2515 -> CAN:AOC346_MCP2515_Holes0.9
- U2: footprint MH_Sensor:MH_Sensor -> MH_Sensor:MH_Sensor_Holes0.9
- U3: footprint RelayModule:Relay_Module_1_Channel -> RelayModule:Relay_Module_1_Channel_Holes0.9
Changed lines of the file:
@@
 F 0 "A1" H 4850 1750 50  0000 C CNN
 F 1 "Arduino_Nano" H 5050 1650 50  0000 C CNN
-F 2 "Module:Arduino_Nano" H 4700 1800 50  0001 L CNN
+F 2 "Arduino:Arduino_Nano_Holes0.9" H 4700 1800 50  0001 L CNN
 F 3 "http://www.mouser.com/pdfdocs/Gravitech_Arduino_Nano3_0.pdf" H 4550 1750 50  0001 C CNN
 	1    4550 2750
@@
 F 0 "U1" H 7600 3128 50  0000 C CNN
 F 1 "MCP2515-TJA1050" H 7600 3037 50  0000 C CNN
-F 2 "CAN:AOC346_MCP2515" H 7600 1450 50  0001 C CIN
+F 2 "CAN:AOC346_MCP2515_Holes0.9" H 7600 1450 50  0001 C CIN
 F 3 "http://arduino.ua/prod1347-modyl-can-shini-na-mcp2515-i-tja1050" H 7700 1550 50  0001 C CNN
 	1    7600 2350
@@
 F 0 "U2" H 6600 1525 50  0000 C CNN
 F 1 "MH-Series" H 6600 1434 50  0000 C CNN
-F 2 "MH_Sensor:MH_Sensor" H 6600 750 50  0001 C CNN
+F 2 "MH_Sensor:MH_Sensor_Holes0.9" H 6600 750 50  0001 C CNN
 F 3 "https://ru.aliexpress.com/item/1pcs-lot-soil-the-hygrometer-detection-module-soil-moisture-sensor-Robot-smart-car/32826425650.html?spm=a2g0v.10010108.1000016.1.7ca9471dkqoaPU&isOrigTitle=true" H 6500 1150 50  0001 C CNN
 	1    6600 1150
@@
 F 0 "U3" H 2950 3150 50  0000 C CNN
 F 1 "5V_Relay_Module" H 2950 3050 50  0000 C CNN
-F 2 "RelayModule:Relay_Module_1_Channel" H 2950 2800 50  0001 C CNN
+F 2 "RelayModule:Relay_Module_1_Channel_Holes0.9" H 2950 2800 50  0001 C CNN
 F 3 "http://arduino.ua/prod2888-modyl-rele-5v-10a-visokogo-yrovnya-high-level" H 2950 2800 50  0001 C CNN
 	1    2950 2800
