File: Schematic/Borjomi-Main.kicad_pcb (KiCad board)
At the start: 2 copper layers, 111.3 x 68.8 mm, 14 parts, among them J1 Vin 12V, J2 Gate 220V, J3 Vout 12V, J4 Data, J5 Pressure, U1 CAN_Module, U2 CurrentMeas_12V, U3 Relay_12Vout, U4 Relay_Gate220V, U5 Bluetooth

Commit message: v1.1. Fix bug with voltage divider
Also update gerber/drill files
Routing:
- net Net-(A1-Pad21): track 91.9 -> 92.5 mm
Changed lines of the file:
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@@
     (thickness 1.6)
     (drawings 25)
-    (tracks 155)
+    (tracks 156)
     (zones 0)
     (modules 14)
@@
   (page A4)
   (layers
-    (0 F.Cu signal)
+    (0 F.Cu signal hide)
     (31 B.Cu signal)
     (32 B.Adhes user hide)
@@
   )
   (setup
-    (last_trace_width 1)
+    (last_trace_width 0.25)
     (user_trace_width 0.2)
     (user_trace_width 0.3)
@@
       (drillshape 0)
       (scaleselection 1)
-      (outputdirectory "gerber/main-v1.0/"))
+      (outputdirectory "gerber/main-v1.1/"))
   )
   (net 0 "")
@@
     (uvia_drill 0.1)
     (add_net GND)
-    (add_net "Net-(A1-Pad1)")
     (add_net "Net-(A1-Pad10)")
-    (add_net "Net-(A1-Pad11)")
     (add_net "Net-(A1-Pad12)")
     (add_net "Net-(A1-Pad13)")
@@
     (add_net "Net-(A1-Pad15)")
     (add_net "Net-(A1-Pad16)")
-    (add_net "Net-(A1-Pad17)")
-    (add_net "Net-(A1-Pad18)")
     (add_net "Net-(A1-Pad19)")
-    (add_net "Net-(A1-Pad2)")
-    (add_net "Net-(A1-Pad20)")
     (add_net "Net-(A1-Pad21)")
-    (add_net "Net-(A1-Pad22)")
     (add_net "Net-(A1-Pad23)")
-    (add_net "Net-(A1-Pad24)")
-    (add_net "Net-(A1-Pad25)")
-    (add_net "Net-(A1-Pad26)")
     (add_net "Net-(A1-Pad27)")
-    (add_net "Net-(A1-Pad28)")
-    (add_net "Net-(A1-Pad3)")
-    (add_net "Net-(A1-Pad30)")
-    (add_net "Net-(A1-Pad5)")
     (add_net "Net-(A1-Pad6)")
     (add_net "Net-(A1-Pad7)")
     (add_net "Net-(A1-Pad8)")
-    (add_net "Net-(A1-Pad9)")
     (add_net "Net-(D1-Pad1)")
     (add_net "Net-(J1-Pad1)")
-    (add_net "Net-(J1-Pad3)")
     (add_net "Net-(J3-Pad2)")
     (add_net "Net-(J4-Pad1)")
     (add_net "Net-(J4-Pad2)")
-    (add_net "Net-(J5-Pad4)")
     (add_net "Net-(U2-Pad5)")
-    (add_net "Net-(U3-Pad6)")
-    (add_net "Net-(U4-Pad6)")
-    (add_net "Net-(U5-Pad1)")
-    (add_net "Net-(U5-Pad6)")
   )
   (module Connector_BarrelJack:BarrelJack_Horizontal (layer F.Cu)
@@
   (segment (start 144.43202 82.7857) (end 141.84122 82.7857) (width 1) (layer B.Cu) (net 2))
   (segment (start 149.99716 94.79534) (end 149.57298 94.37116) (width 0.25) (layer F.Cu) (net 3))
-  (segment (start 155.68422 94.79534) (end 149.99716 94.79534) (width 0.25) (layer F.Cu) (net 3))
   (segment (start 187.452 120.904) (end 188.976 120.904) (width 0.3) (layer B.Cu) (net 3))
   (segment (start 185.547 118.999) (end 187.452 120.904) (width 0.3) (layer B.Cu) (net 3))
@@
   (segment (start 175.006 90.805) (end 184.638001 81.172999) (width 0.3) (layer B.Cu) (net 3))
   (segment (start 191.77 82.423) (end 191.77 90.805) (width 0.3) (layer B.Cu) (net 3))
+  (segment (start 149.99716 94.79534) (end 149.57298 94.37116) (width 0.3) (layer B.Cu) (net 3))
+  (segment (start 155.68422 94.79534) (end 149.99716 94.79534) (width 0.3) (layer B.Cu) (net 3))
   (segment (start 171.831 110.744) (end 173.736 110.744) (width 0.3) (layer B.Cu) (net 4))
   (segment (start 156.718 125.857) (end 171.831 110.744) (width 0.3) (layer B.Cu) (net 4))

Commit message: Update pcb for Borjomi-main
Other:
- board text added: "Borjomi Main v1.1"
- board text removed: "Borjomi Main v1.0"
Changed lines of the file:
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@@
   (gr_line (start 133.731 78.105) (end 142.28318 78.105) (layer B.Mask) (width 2))
   (gr_line (start 144.43202 88.7857) (end 144.43202 94.39402) (layer B.Mask) (width 2))
-  (gr_text "Borjomi\nMain\nv1.0" (at 162.88258 102.34676) (layer F.SilkS)
+  (gr_text "Borjomi\nMain\nv1.1" (at 162.88258 102.34676) (layer F.SilkS)
     (effects (font (size 2 2) (thickness 0.3)))
   )

Commit message: Board Borjomi-Main v1.1 with Gerber/Drill files
Parts:
- added J6: LaptopSwitch, Connector:RJ14_YH-57-21_5722_6P4C, F.Cu at (103.0, 91.6)
- added JP1: Jumper, Connector:SimpleJumper_Pitch5.08mm_Drill0.7mm_2pad, F.Cu at (176.9, 109.5)
- added U6: Relay_LaptopSwitch, RelayModule:Relay_Module_1_Channel_Holes0.9, F.Cu at (100.6, 118.9)
- moved J4 0.50 mm to (219.3, 91.6)
- moved J5 0.50 mm to (202.9, 91.6)
Connections:
- A1 pad 11: (no net) -> Net-(A1-Pad11)
Routing:
- net Net-(JP1-Pad1): track 0.00 -> 85.2 mm
- net Net-(A1-Pad27): track 203.8 -> 233.3 mm
- net Net-(J6-Pad3): track 0.00 -> 17.9 mm
- net Net-(A1-Pad11): track 0.00 -> 13.2 mm
- net Net-(J6-Pad2): track 0.00 -> 12.5 mm
- net Net-(J4-Pad2): track 23.7 -> 24.2 mm
- net Net-(J4-Pad1): track 27.2 -> 27.7 mm
Other:
- board size 111.3 x 68.8 mm -> 132.3 x 68.8 mm
- board text added: "Laptop"
